File: hardware/radio.kicad_pcb (KiCad board)
At the start: 4 copper layers, 115 x 35 mm, 56 parts, among them J101 Cortex_Debug, J102 JAE_DX07S016JA3, J201 SJ2-25404B-SMT-TR, J301 SJ2-25404B-SMT-TR, SW101 SW_Push, SW102 SW_Push, U101 TPS78433QWDRBRQ1, U102 ATSAMD51G, U103 E62, U201 74AHC1G125, U301 TLP2361, Y101 32k768

Commit message: Refresh
Parts:
- renumbered C103 to C102, C104 to C103, C105 to C104, C106 to C105, C107 to C106, C108 to C107, C109 to C108, C110 to C109, C111 to C110, C303 to C111

Commit message: Replace Order_Number
Parts:
- removed C110: 0u1, Capacitor_SMD:C_0603_1608Metric
- removed R102: 1M, Resistor_SMD:R_0603_1608Metric
- C101, C102, C103, C104, C105, C108, C109, C301, C302: footprint Capacitor_SMD:C_0603_1608Metric -> V2_Capacitor_SMD:C_0603
- C106, C107: footprint Capacitor_SMD:C_0603_1608Metric -> V2_Capacitor_SMD:C_0805
- C111: footprint Capacitor_SMD:C_1210_3225Metric -> V2_Capacitor_SMD:C_1210
- D103: footprint LED_SMD:LED_0603_1608Metric -> V2_LED:LED_0603
- D201, D301: footprint Diode_SMD:D_SOD-523 -> V2_Diode_SMD:D_SOD-523
- FID101, FID102, FID103: value Fiducial -> Fiducial_Paste
- H101, H102, H103, H104: value MountingHole_3mm -> 3mm
- INFO102: value ORDER-NUMBER -> ~; footprint V2_Production:Order_Number -> V2_Production:Revision
- J101: value Cortex_Debug -> Cortex; footprint V2_Cortex_Debug:Cortex_Debug_Pad -> V2_Connector_Debug:Cortex
- J102: value JAE_DX07S016JA3 -> DX07S016JA3
- R101, R103, R104, R105, R201, R202, R301: footprint Resistor_SMD:R_0603_1608Metric -> V2_Resistor_SMD:R_0603
- SW101, SW102: value SW_Push -> SKSG
- TVS101, TVS201: footprint Diode_SMD:D_0603_1608Metric -> V2_Diode_SMD:D_0603
- U201: footprint Package_TO_SOT_SMD:SOT-23-5 -> V2_Package_TO_SOT_SMD:SOT-23-5
- U301: footprint Package_SO:SO-5-6_4.55x3.7mm_P1.27mm -> V2_Package_SO:SO-5-6_4.55x3.7mm_P1.27mm
- moved INFO102 24.2 mm to (148.0, 113.5), turned to 0 degrees
- moved C106 0.25 mm to (137.8, 110.2)
- moved C107 0.25 mm to (137.8, 103.8)
- moved TVS101 0.25 mm to (137.8, 112.2)
Connections:
- J102 pad S: Earth -> Shield
Routing:
- net Earth: track 4.39 -> 0.00 mm
- net GND: track 39.9 -> 39.0 mm, vias 47 -> 43
- net +3V3: track 17.9 -> 18.4 mm, vias 9 -> 8
- added copper zone on F.Cu, net Shield
- removed copper zone on F.Cu, net Earth
- removed copper zone on B.Cu, net GND

Commit message: Update Library
Parts:
- C111: value 22u -> 10u
Changed lines of the file:
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@@
 			)
 		)
-		(property "Value" "22u"
+		(property "Value" "10u"
 			(at 0 2.3 270)
 			(layer "F.Fab")

Commit message: Update ESD suppressor
Parts:
- C111: value 10u -> 22u

Commit message: Replace diode
Parts:
- D201, D301: value RB501SM -> PMEG2010EPK; footprint V2_Diode_SMD:D_SOD-523 -> V2_Diode_SMD:D_SOD-1608
Connections:
- net Shield renamed /Shield

Commit message: Update
Parts:
- added C201: 0u1, V2_Capacitor_SMD:C_0603, F.Cu at (142.5, 85.5)
- renumbered C108 to C101, C109 to C102, C101 to C103, C111 to C104, C102 to C105, C103 to C106, C104 to C107, C105 to C108, C106 to C109, C107 to C110, C302 to C301, C301 to C302, D103 to D101, D101 to D102, D102 to D103, INFO102 to INFO101, INFO101 to INFO102, R105 to R101, R101 to R102, R202 to R201, R201 to R202, SW102 to SW101, SW101 to SW102, U103 to U101, U101 to U103
Connections:
- net /VDDCORE renamed /+VCORE
Routing:
- net +5V: track 20.9 -> 22.6 mm
- net GND: track 39.3 -> 39.9 mm, vias 43 -> 44
