File: hardware/radio.kicad_sch (KiCad schematic)
At the start: 42 parts, among them J101 Cortex, J102 DX07S016JA3, SW101 SKSG, SW102 SKSG, U101 TPS78433QWDRBRQ1, U102 ATSAMD51G, U103 E62, Y101 32k768

Commit message: Update
Parts:
- C101: renamed from C108; Id (none) -> Capacitor:${SYMBOL_NAME}; Rating (none) -> 50V
- C102: renamed from C109; Id (none) -> Capacitor:${SYMBOL_NAME}; Rating (none) -> 50V
- C103: renamed from C101; Id (none) -> Capacitor:${SYMBOL_NAME}
- C104: renamed from C111; Id (none) -> Capacitor:${SYMBOL_NAME}
- C105: renamed from C102; Id (none) -> Capacitor:${SYMBOL_NAME}
- C106: renamed from C103; Id (none) -> Capacitor:${SYMBOL_NAME}
- C107: renamed from C104; Id (none) -> Capacitor:${SYMBOL_NAME}
- C108: renamed from C105; Id (none) -> Capacitor:${SYMBOL_NAME}
- C109: renamed from C106; Id (none) -> Capacitor:${SYMBOL_NAME}
- C110: renamed from C107; Id (none) -> Capacitor:${SYMBOL_NAME}
- D101: renamed from D103; Id (none) -> LED:${SYMBOL_NAME}; Rating (none) -> 605nm
- D102: renamed from D101; Id (none) -> LED:${SYMBOL_NAME}; Rating (none) -> 15mA
- D103: renamed from D102; Id (none) -> LED:${SYMBOL_NAME}; Rating (none) -> 15mA
- ESD101: Id (none) -> ESD:${SYMBOL_NAME}; Rating (none) -> 20kV
- J102: Id (none) -> USB:${SYMBOL_NAME}; Rating (none) -> USB2.0
- R101: renamed from R105; Id (none) -> Resistor:${SYMBOL_NAME}
- R102: renamed from R101; Id (none) -> Resistor:${SYMBOL_NAME}
- R103, R104: Id (none) -> Resistor:${SYMBOL_NAME}
- SPACER101, SPACER102, SPACER103, SPACER104: Id (none) -> Spacer:${SYMBOL_NAME}; Manufacturer (none) -> Wurth Elektronik; Mouser (none) -> 710-9774030243R; Product (none) -> 9774030243R; Rating (none) -> 3mm
- SW101: renamed from SW102; Id (none) -> Button:${SYMBOL_NAME}; Rating (none) -> 1.6N
- SW102: renamed from SW101; Id (none) -> Button:${SYMBOL_NAME}; Rating (none) -> 1.6N
- TVS101: Id (none) -> Diode:${SYMBOL_NAME}
- U101: renamed from U103; Id (none) -> Radio:${SYMBOL_NAME}; Manufacturer (none) -> Ebyte Electronic Technology; Product (none) -> E62-433T20S; Rating (none) -> 433Mhz
- U102: Id (none) -> MCU:${SYMBOL_NAME}; Rating (none) -> Cortex-M4F
- U103: renamed from U101; Id (none) -> LDO:${SYMBOL_NAME}; Rating (none) -> 300mA
- Y101: Id (none) -> Crystal:${SYMBOL_NAME}; Rating (none) -> 10ppm
- renumbered INFO102 to INFO101, INFO101 to INFO102
Connections:
- net VDDCORE renamed +VCORE

Commit message: Good Bye Imperial
Parts:
- C101, C102: footprint V2_Capacitor_SMD:C_0603 -> V2_Capacitor_SMD:C_1608; symbol V2_Capacitor:0603_18p -> V2_Capacitor:1608_18p
- C103: footprint V2_Capacitor_SMD:C_0603 -> V2_Capacitor_SMD:C_1608; symbol V2_Capacitor:0603_10u -> V2_Capacitor:1608_10u
- C104: footprint V2_Capacitor_SMD:C_1210 -> V2_Capacitor_SMD:C_3225; symbol V2_Capacitor:1210_22u -> V2_Capacitor:3225_22u
- C105, C106, C107, C108: footprint V2_Capacitor_SMD:C_0603 -> V2_Capacitor_SMD:C_1608; symbol V2_Capacitor:0603_0u1 -> V2_Capacitor:1608_0u1
- C109, C110: footprint V2_Capacitor_SMD:C_0805 -> V2_Capacitor_SMD:C_2012; symbol V2_Capacitor:0805_10u -> V2_Capacitor:2012_10u
- D101: symbol V2_LED:0603_Orange -> V2_LED:1608_Orange
- R101: footprint V2_Resistor_SMD:R_0603 -> V2_Resistor_SMD:R_1608; symbol V2_Resistor:0603_100k -> V2_Resistor:1608_100k
- R102: footprint V2_Resistor_SMD:R_0603 -> V2_Resistor_SMD:R_1608; symbol V2_Resistor:0603_330R -> V2_Resistor:1608_330R
- R103, R104: footprint V2_Resistor_SMD:R_0603 -> V2_Resistor_SMD:R_1608; symbol V2_Resistor:0603_5k1 -> V2_Resistor:1608_5k1
Changed lines of the file:
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@@
 	)
 	(symbol
-		(lib_id "V2_Capacitor:0603_0u1")
+		(lib_id "V2_Capacitor:1608_0u1")
 		(at 115.57 25.4 0)
 		(unit 1)
@@
 			)
 		)
-		(property "Footprint" "V2_Capacitor_SMD:C_0603"
+		(property "Footprint" "V2_Capacitor_SMD:C_1608"
 			(at 115.57 42.418 0)
 			(hide yes)
@@
 	)
 	(symbol
-		(lib_id "V2_LED:0603_Orange")
+		(lib_id "V2_LED:1608_Orange")
 		(at 125.73 59.69 0)
 		(mirror y)
@@
 	)
 	(symbol
-		(lib_id "V2_Capacitor:0805_10u")
+		(lib_id "V2_Capacitor:2012_10u")
 		(at 201.93 39.37 0)
 		(unit 1)
@@
 			)
 		)
-		(property "Footprint" "V2_Capacitor_SMD:C_0805"
+		(property "Footprint" "V2_Capacitor_SMD:C_2012"
 			(at 201.93 56.388 0)
 			(hide yes)
@@
 	)
 	(symbol
-		(lib_id "V2_Resistor:0603_5k1")
+		(lib_id "V2_Resistor:1608_5k1")
 		(at 219.71 97.79 90)
 		(unit 1)
@@
 			)
 		)
-		(property "Footprint" "V2_Resistor_SMD:R_0603"
+		(property "Footprint" "V2_Resistor_SMD:R_1608"
 			(at 235.458 97.79 0)
 			(hide yes)
@@
 	)
 	(symbol
-		(lib_id "V2_Capacitor:1210_22u")
+		(lib_id "V2_Capacitor:3225_22u")
 		(at 72.39 170.18 0)
 		(unit 1)
@@
 			)
 		)
-		(property "Footprint" "V2_Capacitor_SMD:C_1210"
+		(property "Footprint" "V2_Capacitor_SMD:C_3225"
 			(at 72.39 187.198 0)
 			(hide yes)
@@
 	)
 	(symbol
-		(lib_id "V2_Capacitor:0805_10u")
+		(lib_id "V2_Capacitor:2012_10u")
 		(at 175.26 39.37 0)
 		(unit 1)
@@
 			)
 		)
-		(property "Footprint" "V2_Capacitor_SMD:C_0805"
+		(property "Footprint" "V2_Capacitor_SMD:C_2012"
 			(at 175.26 56.388 0)
 			(hide yes)
@@
 	)
 	(symbol
-		(lib_id "V2_Capacitor:0603_18p")
+		(lib_id "V2_Capacitor:1608_18p")
 		(at 31.75 48.26 0)
 		(unit 1)
@@
 			)
 		)
-		(property "Footprint" "V2_Capacitor_SMD:C_0603"
+		(property "Footprint" "V2_Capacitor_SMD:C_1608"
 			(at 31.75 65.278 0)
 			(hide yes)
@@
 	)
 	(symbol
-		(lib_id "V2_Capacitor:0603_10u")
+		(lib_id "V2_Capacitor:1608_10u")
 		(at 64.77 25.4 0)
 		(unit 1)
@@
 			)
 		)
-		(property "Footprint" "V2_Capacitor_SMD:C_0603"
+		(property "Footprint" "V2_Capacitor_SMD:C_1608"
 			(at 64.77 42.418 0)
 			(hide yes)
@@
 	)
 	(symbol
-		(lib_id "V2_Capacitor:0603_18p")
+		(lib_id "V2_Capacitor:1608_18p")
 		(at 26.67 48.26 0)
 		(unit 1)
@@
 			)
 		)
-		(property "Footprint" "V2_Capacitor_SMD:C_0603"
+		(property "Footprint" "V2_Capacitor_SMD:C_1608"
 			(at 26.67 65.278 0)
 			(hide yes)
@@
 	)
 	(symbol
-		(lib_id "V2_Resistor:0603_330R")
+		(lib_id "V2_Resistor:1608_330R")
 		(at 135.89 59.69 90)
 		(unit 1)
@@
 			)
 		)
-		(property "Footprint" "V2_Resistor_SMD:R_0603"
+		(property "Footprint" "V2_Resistor_SMD:R_1608"
 			(at 151.638 59.69 0)
 			(hide yes)
@@
 	)
 	(symbol
-		(lib_id "V2_Capacitor:0603_0u1")
+		(lib_id "V2_Capacitor:1608_0u1")
 		(at 105.41 25.4 0)
 		(unit 1)
@@
 			)
 		)
-		(property "Footprint" "V2_Capacitor_SMD:C_0603"
+		(property "Footprint" "V2_Capacitor_SMD:C_1608"
 			(at 105.41 42.418 0)
 			(hide yes)
@@
 	)
 	(symbol
-		(lib_id "V2_Capacitor:0603_0u1")
+		(lib_id "V2_Capacitor:1608_0u1")
 		(at 85.09 25.4 0)
 		(unit 1)
@@
 			)
 		)
-		(property "Footprint" "V2_Capacitor_SMD:C_0603"
+		(property "Footprint" "V2_Capacitor_SMD:C_1608"
 			(at 85.09 42.418 0)
 			(hide yes)
@@
 	)
 	(symbol
-		(lib_id "V2_Capacitor:0603_0u1")
+		(lib_id "V2_Capacitor:1608_0u1")
 		(at 95.25 25.4 0)
 		(unit 1)
@@
 			)
 		)
-		(property "Footprint" "V2_Capacitor_SMD:C_0603"
+		(property "Footprint" "V2_Capacitor_SMD:C_1608"
 			(at 95.25 42.418 0)
 			(hide yes)
@@
 	)
 	(symbol
-		(lib_id "V2_Resistor:0603_5k1")
+		(lib_id "V2_Resistor:1608_5k1")
 		(at 219.71 95.25 90)
 		(unit 1)
@@
 			)
 		)
-		(property "Footprint" "V2_Resistor_SMD:R_0603"
+		(property "Footprint" "V2_Resistor_SMD:R_1608"
 			(at 235.458 95.25 0)
 			(hide yes)
@@
 	)
 	(symbol
-		(lib_id "V2_Resistor:0603_100k")
+		(lib_id "V2_Resistor:1608_100k")
 		(at 57.15 123.19 90)
 		(unit 1)
@@
 			)
 		)
-		(property "Footprint" "V2_Resistor_SMD:R_0603"
+		(property "Footprint" "V2_Resistor_SMD:R_1608"
 			(at 72.898 123.19 0)
 			(hide yes)
